Commit message: trials

File: rrbot_description/urdf/fullGoatLeg.xacro (robot description, xacro)
@@ -8,10 +8,10 @@
   <!-- Import Rviz colors -->
 	<xacro:include filename="$(find rrbot_description)/urdf/openGoatLeg.xacro" />
-	<link name="world" />
+<!-- 	<link name="world" />
 	<joint name="world_joint" type="fixed">
 		<parent link="world" />
 		<child link = "hipJoint" />
 		<origin xyz="0.0 0.0 1" rpy="0.0 0.0 0.0" />
-	</joint>
+	</joint> -->
 	<link name="footAssembly">
 		<visual>
@@ -19,5 +19,5 @@
 				<mesh filename="package://rrbot_description/meshes/footassembly.dae"/>
 			</geometry>
-			<origin xyz="0 0 0" rpy="0 0 ${PI}"/>
+			<origin xyz="0 0 0" rpy="0 0 3.1415926535897931"/>
 		</visual>
 		<collision>
@@ -25,5 +25,5 @@
 				<mesh filename="package://rrbot_description/meshes/footassembly.dae"/>
 			</geometry>
-			<origin xyz="0 0 0" rpy="0 0 ${PI}"/>
+			<origin xyz="0 0 0" rpy="0 0 3.1415926535897931"/>
 		</collision>
 		<inertial>
@@ -32,10 +32,17 @@
 		</inertial>
   	</link>
-  	<joint name="footBracket_to_footAssembly" type="revolute">
+  	<joint name="footAssembly_to_leg1_footBracket" type="revolute">
 		<axis xyz="0 0 1"/>
-		<limit effort="1000.0" lower="${-PI}" upper="${PI}" velocity="0"/>
+		<limit effort="1000.0" lower="-3.1415926535897931" upper="3.1415926535897931" velocity="0"/>
 		<origin xyz="0 0.01159 0" rpy="0 0 0"/>
+		<child link="footAssembly"/>
 		<parent link="leg1_footBracket"/>
-		<child link="leg2_footBracket"/>
   	</joint>
+  	<!-- <joint name="footAssembly_to_leg2_footBracket" type="revolute">
+		<axis xyz="0 0 1"/>
+		<limit effort="1000.0" lower="-3.1415926535897931" upper="3.1415926535897931" velocity="0"/>
+		<origin xyz="0 0.01159 0" rpy="0 0 0"/>
+		<child link="footAssembly"/>
+		<parent link="leg2_footBracket"/>
+  	</joint> -->
 </robot>

File: rrbot_description/urdf/openGoatLeg.xacro (robot description, xacro)
@@ -306,4 +306,29 @@
 <xacro:singleLeg prefix="leg2" reflect="1" />
 <xacro:singleLeg prefix="leg3" reflect="2" />
+<!--   <link name="footAssembly">
+    <visual>
+      <geometry>
+        <mesh filename="package://rrbot_description/meshes/footassembly.dae"/>
+      </geometry>
+      <origin xyz="0 0 0" rpy="0 0 3.1415926535897931"/>
+    </visual>
+    <collision>
+      <geometry>
+        <mesh filename="package://rrbot_description/meshes/footassembly.dae"/>
+      </geometry>
+      <origin xyz="0 0 0" rpy="0 0 3.1415926535897931"/>
+    </collision>
+    <inertial>
+      <mass value="0.02883033104"/>
+      <inertia ixx="0.00757" ixy="0.0" ixz="0.0" iyy="0.212" iyz="0.0" izz="0.21199"/>
+    </inertial>
+  </link>
+  <joint name="footAssembly_to_leg1_footBracket" type="revolute">
+    <axis xyz="0 0 1"/>
+    <limit effort="1000.0" lower="-3.1415926535897931" upper="3.1415926535897931" velocity="0"/>
+    <origin xyz="0 0.01159 0" rpy="0 0 0"/>
+    <child link="footAssembly"/>
+    <parent link="leg1_footBracket"/>
+  </joint> -->
   <!-- GAZEBO PLUGIN -->
 <!-- <gazebo>

File: rrbot_description/urdf/singleLeg.urdf (robot description, URDF)
Before this commit: robot rrbot, 2 links, 1 joints
Links:
- added link hipJoint, mass 0.02883033104; collision mesh filename=package://rrbot_description/meshes/singleleghipjoint.dae; visual mesh filename=package://rrbot_description/meshes/singleleghipjoint.dae
- added link leg1_bendElbow, mass 0.02883033104; collision mesh filename=package://rrbot_description/meshes/elbow_bend.dae; visual mesh filename=package://rrbot_description/meshes/elbow_bend.dae
- added link leg1_eyeJoint, mass 0.02883033104; collision mesh filename=package://rrbot_description/rrbot_description/meshes/eye_jo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; visual mesh filename=package://rrbot_description/meshes/eye_joint.dae
- added link leg1_footBracket, mass 0.02883033104; collision mesh filename=package://rrbot_description/meshes/foot_bracket.dae; visual mesh filename=package://rrbot_description/meshes/foot_bracket.dae
- added link leg1_lowerLeg, mass 0.02883033104; collision mesh filename=package://rrbot_description/meshes/lower_leg.dae; visual mesh filename=package://rrbot_description/meshes/lower_leg.dae
- added link leg1_sphericalJointMiddleLink, mass 0.02883033104; collision mesh filename=package://rrbot_description/meshes/spherical_joint_middle_p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; visual mesh filename=package://rrbot_description/meshes/spherical_joint_middle_p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
- added link leg1_upper_leg, mass 0.02883033104; collision mesh filename=package://rrbot_description/meshes/upper_leg.dae; visual mesh filename=package://rrbot_description/meshes/upper_leg.dae
- added link leg1_upper_leg_bracket, mass 0.02883033104; collision mesh filename=package://rrbot_description/meshes/upper_leg_bracket.dae; visual mesh filename=package://rrbot_description/meshes/upper_leg_bracket.dae
- added link leg2_bendElbow, mass 0.02883033104; collision mesh filename=package://rrbot_description/meshes/elbow_bend.dae; visual mesh filename=package://rrbot_description/meshes/elbow_bend.dae
- added link leg2_eyeJoint, mass 0.02883033104; collision mesh filename=package://rrbot_description/meshes/eye_joint.dae; visual mesh filename=package://rrbot_description/meshes/eye_joint.dae
- added link leg2_footBracket, mass 0.02883033104; collision mesh filename=package://rrbot_description/meshes/foot_bracket.dae; visual mesh filename=package://rrbot_description/meshes/foot_bracket.dae
- added link leg2_lowerLeg, mass 0.02883033104; collision mesh filename=package://rrbot_description/meshes/lower_leg.dae; visual mesh filename=package://rrbot_description/meshes/lower_leg.dae
- added link leg2_motormountingbracket_fixed, mass 0.02883033104; collision mesh filename=package://rrbot_description/meshes/motormountingbracket_fix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; visual mesh filename=package://rrbot_description/meshes/motormountingbracket_fix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
- added link leg2_pipebetweenhipandmotormountingbracket, mass 0.02883033104; collision mesh filename=package://rrbot_description/meshes/pipebetweenhipandmotormo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; visual mesh filename=package://rrbot_description/meshes/pipebetweenhipandmotormo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
- added link leg2_sphericalJointMiddleLink, mass 0.02883033104; collision mesh filename=package://rrbot_description/meshes/spherical_joint_middle_p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; visual mesh filename=package://rrbot_description/meshes/spherical_joint_middle_p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
- added link leg2_upper_leg, mass 0.02883033104; collision mesh filename=package://rrbot_description/meshes/upper_leg.dae; visual mesh filename=package://rrbot_description/meshes/upper_leg.dae
- added link leg2_upper_leg_bracket, mass 0.02883033104; collision mesh filename=package://rrbot_description/meshes/upper_leg_bracket.dae; visual mesh filename=package://rrbot_description/meshes/upper_leg_bracket.dae
- added link leg3_bendElbow, mass 0.02883033104; collision mesh filename=package://rrbot_description/meshes/elbow_bend.dae; visual mesh filename=package://rrbot_description/meshes/elbow_bend.dae
- added link leg3_eyeJoint, mass 0.02883033104; collision mesh filename=package://rrbot_description/meshes/eye_joint.dae; visual mesh filename=package://rrbot_description/meshes/eye_joint.dae
- added link leg3_footBracket, mass 0.02883033104; collision mesh filename=package://rrbot_description/meshes/foot_bracket.dae; visual mesh filename=package://rrbot_description/meshes/foot_bracket.dae
- added link leg3_lowerLeg, mass 0.02883033104; collision mesh filename=package://rrbot_description/meshes/lower_leg.dae; visual mesh filename=package://rrbot_description/meshes/lower_leg.dae
- added link leg3_motormountingbracket_fixed, mass 0.02883033104; collision mesh filename=package://rrbot_description/meshes/motormountingbracket_fix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; visual mesh filename=package://rrbot_description/meshes/motormountingbracket_fix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
- added link leg3_pipebetweenhipandmotormountingbracket, mass 0.02883033104; collision mesh filename=package://rrbot_description/meshes/pipebetweenhipandmotormo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; visual mesh filename=package://rrbot_description/meshes/pipebetweenhipandmotormo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
- added link leg3_sphericalJointMiddleLink, mass 0.02883033104; collision mesh filename=package://rrbot_description/meshes/spherical_joint_middle_p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; visual mesh filename=package://rrbot_description/meshes/spherical_joint_middle_p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
- added link leg3_upper_leg, mass 0.02883033104; collision mesh filename=package://rrbot_description/meshes/upper_leg.dae; visual mesh filename=package://rrbot_description/meshes/upper_leg.dae
- added link leg3_upper_leg_bracket, mass 0.02883033104; collision mesh filename=package://rrbot_description/meshes/upper_leg_bracket.dae; visual mesh filename=package://rrbot_description/meshes/upper_leg_bracket.dae
- added link world
Joints:
- added joint fixed: type fixed, parent world, child hipJoint, origin xyz=0 0 1 rpy=0 0 0
- added joint leg1_bendElbow_to_lowerLeg: type fixed, parent leg1_bendElbow, child leg1_lowerLeg, origin xyz=0.06170 0.01192 0 rpy=0 0 0.820304748
- added joint leg1_eyeJoint_to_sphericalJointMiddleLink: type revolute, parent leg1_eyeJoint, child leg1_sphericalJointMiddleLink, origin xyz=0 0 0 rpy=0 0 0, axis 0 0 1, limit lower=-1.570796327 upper=1.570796327 effort=1000.0 velocity=0
- added joint leg1_hip_to_pipeBetweenHipAndMotorMountingBracket: type fixed, parent hipJoint, child leg1_pipebetweenhipandmotormountingbracket, origin xyz=0.01176 0  0 rpy=0 0 0
- added joint leg1_lowerLeg_footBracket: type fixed, parent leg1_lowerLeg, child leg1_footBracket, origin xyz=0.26032 0 0 rpy=0 0 0
- added joint leg1_motorMoutingBracket_to_upperLegBracket: type revolute, parent leg1_motormountingbracket_fixed, child leg1_upper_leg_bracket, origin xyz=0.00864 0.06680 0.01267 rpy=0 0 0, axis 0 0 1, limit lower=-1.570796327 upper=1.570796327 effort=1000.0 velocity=0
- added joint leg1_sphericalJointMiddleLink_to_bendElbow: type revolute, parent leg1_sphericalJointMiddleLink, child leg1_bendElbow, origin xyz=0.01916 0 0 rpy=0 0 0, axis 1 0 0, limit lower=-3.1415926535897931 upper=3.1415926535897931 effort=1000.0 velocity=0
- added joint leg1_upperLegBracket_to_upperLink: type fixed, parent leg1_upper_leg_bracket, child leg1_upper_leg, origin xyz=0.05166 0 -0.01150 rpy=0 0 0
- added joint leg1_upperLeg_to_eyeJoint: type revolute, parent leg1_upper_leg, child leg1_eyeJoint, origin xyz=0.09885 0 0 rpy=0 0 0, axis 1 0 0, limit lower=-3.1415926535897931 upper=3.1415926535897931 effort=1000.0 velocity=0
- added joint leg2_bendElbow_to_lowerLeg: type fixed, parent leg2_bendElbow, child leg2_lowerLeg, origin xyz=0.06170 0.01192 0 rpy=0 0 0.820304748
- added joint leg2_eyeJoint_to_sphericalJointMiddleLink: type revolute, parent leg2_eyeJoint, child leg2_sphericalJointMiddleLink, origin xyz=0 0 0 rpy=0 0 0, axis 0 0 1, limit lower=-1.570796327 upper=1.570796327 effort=1000.0 velocity=0
- added joint leg2_hip_to_pipeBetweenHipAndMotorMountingBracket: type fixed, parent hipJoint, child leg2_pipebetweenhipandmotormountingbracket, origin xyz=-0.00588 0.0101844587484998  0 rpy=0 0 2.0943951023931955
- added joint leg2_lowerLeg_footBracket: type fixed, parent leg2_lowerLeg, child leg2_footBracket, origin xyz=0.26032 0 0 rpy=0 0 0
- added joint leg2_motorMoutingBracket_to_upperLegBracket: type revolute, parent leg2_motormountingbracket_fixed, child leg2_upper_leg_bracket, origin xyz=0.00864 0.06680 0.01267 rpy=0 0 0, axis 0 0 1, limit lower=-1.570796327 upper=1.570796327 effort=1000.0 velocity=0
- added joint leg2_pipebetweenhipandmotormountingbracket_to_motor: type fixed, parent leg2_pipebetweenhipandmotormountingbracket, child leg2_motormountingbracket_fixed, origin xyz=0.03073 0 0 rpy=-1.570796327 0 0
- added joint leg2_sphericalJointMiddleLink_to_bendElbow: type revolute, parent leg2_sphericalJointMiddleLink, child leg2_bendElbow, origin xyz=0.01916 0 0 rpy=0 0 0, axis 1 0 0, limit lower=-3.1415926535897931 upper=3.1415926535897931 effort=1000.0 velocity=0
- added joint leg2_upperLegBracket_to_upperLink: type fixed, parent leg2_upper_leg_bracket, child leg2_upper_leg, origin xyz=0.05166 0 -0.01150 rpy=0 0 0
- added joint leg2_upperLeg_to_eyeJoint: type revolute, parent leg2_upper_leg, child leg2_eyeJoint, origin xyz=0.09885 0 0 rpy=0 0 0, axis 1 0 0, limit lower=-3.1415926535897931 upper=3.1415926535897931 effort=1000.0 velocity=0
- added joint leg3_bendElbow_to_lowerLeg: type fixed, parent leg3_bendElbow, child leg3_lowerLeg, origin xyz=0.06170 0.01192 0 rpy=0 0 0.820304748
- added joint leg3_eyeJoint_to_sphericalJointMiddleLink: type revolute, parent leg3_eyeJoint, child leg3_sphericalJointMiddleLink, origin xyz=0 0 0 rpy=0 0 0, axis 0 0 1, limit lower=-1.570796327 upper=1.570796327 effort=1000.0 velocity=0
- added joint leg3_hip_to_pipeBetweenHipAndMotorMountingBracket: type fixed, parent hipJoint, child leg3_pipebetweenhipandmotormountingbracket, origin xyz=-0.00588 -0.0101844587484998 0 rpy=0 0 4.188790204786391
- added joint leg3_lowerLeg_footBracket: type fixed, parent leg3_lowerLeg, child leg3_footBracket, origin xyz=0.26032 0 0 rpy=0 0 0
- added joint leg3_motorMoutingBracket_to_upperLegBracket: type revolute, parent leg3_motormountingbracket_fixed, child leg3_upper_leg_bracket, origin xyz=0.00864 0.06680 0.01267 rpy=0 0 0, axis 0 0 1, limit lower=-1.570796327 upper=1.570796327 effort=1000.0 velocity=0
- added joint leg3_pipebetweenhipandmotormountingbracket_to_motor: type fixed, parent leg3_pipebetweenhipandmotormountingbracket, child leg3_motormountingbracket_fixed, origin xyz=0.03073 0 0 rpy=-1.570796327 0 0
- added joint leg3_sphericalJointMiddleLink_to_bendElbow: type revolute, parent leg3_sphericalJointMiddleLink, child leg3_bendElbow, origin xyz=0.01916 0 0 rpy=0 0 0, axis 1 0 0, limit lower=-3.1415926535897931 upper=3.1415926535897931 effort=1000.0 velocity=0
- added joint leg3_upperLegBracket_to_upperLink: type fixed, parent leg3_upper_leg_bracket, child leg3_upper_leg, origin xyz=0.05166 0 -0.01150 rpy=0 0 0
- added joint leg3_upperLeg_to_eyeJoint: type revolute, parent leg3_upper_leg, child leg3_eyeJoint, origin xyz=0.09885 0 0 rpy=0 0 0, axis 1 0 0, limit lower=-3.1415926535897931 upper=3.1415926535897931 effort=1000.0 velocity=0
- joint leg1_pipebetweenhipandmotormountingbracket_to_motor: origin xyz=0.03073 0 0 rpy=-1.570 0 0 -> xyz=0.03073 0 0 rpy=-1.570796327 0 0
